Commit message: uika的himloco训练成功

File: source/moma_lab/moma_lab/data/Robots/uika/uika_description/urdf/uika_simple_collision.urdf (robot description, URDF)
Before this commit: robot UIKA, 17 links, 16 joints
Links:
- added link mid360_link
Joints:
- added joint mid360_joint: type fixed, parent base, child mid360_link, origin xyz=0.33 0 -0.08 rpy=0 2.5 0
